File: aerolotl.kicad_pcb (KiCad board)
At the start: 2 copper layers, 31 parts, among them CN1 StemmaQT, J1 SWD, J6 FTSH-107-STDC14, Q1 AO3400A, Q2 AO3400A, Q3 AO3400A, SW1 SW_Nidec_CAS-120A1, U1 STM32H755ZIT6, U10 LMR51430XFDDCR, U2 BMP581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

Commit message: solved reverse polarity w pmos and tvs clamp
Parts:
- moved U1 14.7 mm to (132.0, 77.0), turned to 45 degrees
